File: hardware/TouchTone555.kicad_pcb (KiCad board)
At the start: 2 copper layers, 200 x 96 mm, 73 parts, among them J1 DC Barrel Jack, J2 9V Battery, J3 PJ-320A, J4 Stylus, J5 Speaker, Q1 BC548, Q2 2N3904, Q3 2N3906, SW1 POWER, SW2 VIBRATO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

Commit message: Fixed values for trim pots & R8
Tuning trim potentiometers were incorrectly listed as 10K, have been changed to 5K.
Vibrato trim potentiometer was incorrectly listed as 250R, has been changed to 10K.
R8 was incorrectly listed as 20K, should be 10K.
Parts:
- R8: value 20K -> 10K
- VR1: value 3296W-1-250 -> 3296W 10K
- VR10, VR11, VR13, VR14, VR15, VR16, VR17, VR18, VR19, VR2, VR20, VR21, VR22, VR3, VR4, VR5, VR6, VR7, VR8, VR9: value 3296W 10K -> 3296W 5K
